File: SMproject_02/KRP_SMproject_02.brd (EAGLE design)
At the start: 160 x 100 mm, 31 parts, among them IC1 STM32F405RGT6, IC2 MCP2561-E_SN, IC3 NJM2845DL1-05-TE1, IC4 NJM78L33SU3, J1 BH-10SG, J2 B5B-EH-A__LF___SN_, Y1 26mhz

Commit message: third
Parts:
- moved IC4 104.2 mm to (20.3, 68.6)
- moved C2 102.4 mm to (21.6, 54.6)
- moved C1 102.4 mm to (17.8, 61.0), turned to 90 degrees
- moved Y1 87.5 mm to (50.8, 81.3), turned to 270 degrees
- moved R3 86.7 mm to (38.1, 59.7)
- moved R4 84.2 mm to (30.5, 59.7)
- moved C14 77.8 mm to (16.5, 81.3), turned to 270 degrees
- moved C12 76.7 mm to (21.6, 81.3), turned to 270 degrees
- moved C19 74.7 mm to (48.3, 67.3)
- moved C6 74.5 mm to (25.4, 81.3), turned to 90 degrees
- moved R2 74.5 mm to (16.5, 86.4), turned to 270 degrees
- moved C10 74.3 mm to (48.3, 73.7)
- moved C9 73.3 mm to (31.8, 86.4)
- moved C16 72.6 mm to (21.6, 86.4), turned to 270 degrees
- moved C5 72.2 mm to (25.4, 86.4), turned to 270 degrees
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Routing:
- net +5V: track 0.00 -> 391.7 mm, vias 0 -> 20
- net GND: track 0.00 -> 391.6 mm, vias 0 -> 7
- net CS: track 0.00 -> 150.1 mm, vias 0 -> 9
- net SDO: track 0.00 -> 137.1 mm, vias 0 -> 4
- net N$3: track 0.00 -> 120.8 mm, vias 0 -> 1
- net SDI: track 0.00 -> 103.6 mm, vias 0 -> 5
- net CK: track 0.00 -> 96.7 mm, vias 0 -> 2
- net N$5: track 0.00 -> 69.9 mm, vias 0 -> 2
- net N$7: track 0.00 -> 59.3 mm, vias 0 -> 2
- net RXD: track 0.00 -> 49.3 mm, vias 0 -> 4
- net N$9: track 0.00 -> 48.2 mm
- net CANL: track 0.00 -> 46.9 mm, vias 0 -> 1
- net CANH: track 0.00 -> 42.7 mm, vias 0 -> 4
- net N$1: track 0.00 -> 42.6 mm
- net TXD: track 0.00 -> 42.3 mm, vias 0 -> 2
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